File: kicad_files/projet.kicad_sch (KiCad schematic)
At the start: 76 parts, among them J1 STLink V3, J2 Sortie, J4 USB_B_Micro, Q1 BC817, Q10 IRLML0030, Q2 BC817, Q3 NMOS, Q4 PMOS, Q5 BC817, Q6 BC817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

Commit message: circuit
Parts:
- removed Q3: NMOS, symbol Simulation_SPICE:NMOS
- removed Q4: PMOS, symbol Simulation_SPICE:PMOS
- added Q3: IRLML0030, Package_TO_SOT_SMD:SOT-23, symbol Transistor_FET:IRLML0030
- added R25: 10k, symbol Device:R
Connections:
- net at U2.8 (Vout), U6.5 (P0A), U6.6 (P0W): now also Q3.2 (S)
- net SORTIE_BYPASS: now reaches J2.1 (Pin_1), U4.6 (-), U4.7
- net SORTIE_BYPASS: now also Q3.3 (D)
- new net BYPASS: Q3.1 (G), R25.2
- no-connect marks 2 -> 19

Commit message: circuit
Parts:
- removed C18: 0.1u, symbol Device:C
- removed C19: 6.8u, symbol Device:C
- removed U5: CD4066BM, Package_SO:SO-14_3.9x8.65mm_P1.27mm, symbol Analog_Switch:CD4066BM

Commit message: circuit
Parts:
- removed Q3: IRLML0030, Package_TO_SOT_SMD:SOT-23, symbol Transistor_FET:IRLML0030
- removed R25: 10k, symbol Device:R
Connections:
- net SORTIE_BYPASS: no longer names the net of J2.1 (Pin_1), U4.6 (-), U4.7

Commit message: circuit
Parts:
- removed R12, R13, R17: 10k, symbol Device:R
Connections:
- net BT1: now also R2.2, SW3.1
- net BT2: now also R4.2, SW4.1
- net BT3: now also R16.2, SW5.1
- net SORTIE_FILTRE: now also C10.1, C15.1, C16.1, C17.1; no longer Q10.3 (D), Q7.3 (D), Q8.3 (D), Q9.3 (D)
- net at Q10.2 (S): no longer C17.1
- net at Q9.2 (S): no longer C16.1
- net at C16.2: now also Q9.3 (D)
- net at Q7.2 (S): no longer C10.1
- net at C10.2: now also Q7.3 (D)
- net at Q8.2 (S): no longer C15.1
- net at C17.2: now also Q10.3 (D)
- net at C15.2: now also Q8.3 (D)
Other:
- moved on the sheet: C10, C15, C16, C17, Q10, Q7, Q8, Q9, R21, R22, R23, R24

Commit message: circuit ok
Parts:
- removed C20: 6.8u, symbol Device:C
- removed C21: 0.1u, symbol Device:C
- removed R18, R19, R20, R7: R, symbol Device:R
- removed U7: TLV2372, symbol Amplifier_Operational:TLV2372
- RV2: value R_Potentiometer -> ~
Connections:
- net SORTIE_FILTRE: now also U4.3 (+)
- net at R5.2: now also C12.1
- no-connect marks 19 -> 16
Other:
- moved on the sheet: C10, C11, C15, C16, C17, C6, C7, J2, Q10, Q7, Q8, Q9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
