File: Applied.kicad_sch (KiCad schematic)
At the start: 62 parts, among them J1 STLink V3, J4 USB_B_Micro, J5 Conn_01x04, Q1 BC817, Q10 IRLML0030, Q2 BC817, Q5 BC817, Q7 IRLML0030, Q8 IRLML0030, Q9 IRLML0030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

Commit message: Add files via upload
final
Connections:
- net +3.3V: no longer C2.1, R3.1, U3.2 (VO)
- net GND2: now reaches J1.4 (Pin_4)
- new net: C2.1, R3.1, U3.2 (VO)
